Commit message: correct joint naming conventions

File: multilink_balancer_description/urdf/multilink_balancer.xacro (robot description, xacro)
@@ -141,5 +141,5 @@
       </inertial>
   </link>
-  <joint name="joint4" type="continuous">
+  <joint name="joint3" type="continuous">
     <parent link="link3"/>
     <child link="link4"/>
@@ -172,5 +172,5 @@
       </inertial>
   </link>
-  <joint name="joint5" type="continuous">
+  <joint name="joint4" type="continuous">
     <parent link="link3"/>
     <child link="link5"/>

Commit message: add ros controllers on new joints

File: multilink_balancer_description/urdf/multilink_balancer.xacro (robot description, xacro)
@@ -224,3 +224,23 @@
     </actuator>
   </transmission>
+  <transmission name="tran3">
+    <type>transmission_interface/SimpleTransmission</type>
+    <joint name="joint3">
+      <hardwareInterface>hardware_interface/EffortJointInterface</hardwareInterface>
+    </joint>
+    <actuator name="motor3">
+      <hardwareInterface>hardware_interface/EffortJointInterface</hardwareInterface>
+      <mechanicalReduction>1</mechanicalReduction>
+    </actuator>
+  </transmission>
+  <transmission name="tran4">
+    <type>transmission_interface/SimpleTransmission</type>
+    <joint name="joint4">
+      <hardwareInterface>hardware_interface/EffortJointInterface</hardwareInterface>
+    </joint>
+    <actuator name="motor4">
+      <hardwareInterface>hardware_interface/EffortJointInterface</hardwareInterface>
+      <mechanicalReduction>1</mechanicalReduction>
+    </actuator>
+  </transmission>
 </robot>

Commit message: match spatial_v2 model exactly

File: multilink_balancer_description/urdf/multilink_balancer.xacro (robot description, xacro)
@@ -13,5 +13,6 @@
   <xacro:property name="foot_height" value="0.05" /> <!-- Foot dimensions -->
   <xacro:property name="foot_width" value="1.0" />
-  <xacro:property name="foot_mass" value="0.2" /> <!-- negligible mass for the foot -->
+  <xacro:property name="foot_mass" value="1.0" /> <!-- negligible mass for the foot -->
+  <xacro:property name="damping" value="0.0" />
   <xacro:property name="axel_offset" value="0.05" /> <!-- How far keep joints away from each other -->
   <!-- Import all Gazebo-customization elements, including Gazebo colors -->
@@ -20,9 +21,10 @@
   <xacro:include filename="$(find multilink_balancer_description)/urdf/materials.xacro" />
   <!-- Used for fixing robot foot to the world -->
+  <!--
   <link name="world"/>
   <joint name="fixed" type="fixed">
     <parent link="world"/>
     <child link="foot"/>
-  </joint>
+  </joint>-->
   <!-- Foot Link-->
   <link name="foot">
@@ -84,5 +86,5 @@
     <origin xyz="0 ${width} ${height1 - axel_offset}" rpy="0 0 0"/>
     <axis xyz="0 1 0"/>
-    <dynamics damping="0.7"/>
+    <dynamics damping="${damping}"/>
   </joint>
   <!-- Bottom Link -->
@@ -105,8 +107,8 @@
       <mass value="${mass}"/>
       <inertia
-          ixx="${mass / 12.0 * (width*width + height2*height2)}" ixy="0.0" ixz="0.0"
-          iyy="${mass / 12.0 * (height2*height2 + width*width)}" iyz="0.0"
-          izz="${mass / 12.0 * (width*width + width*width)}"/>
-      </inertial>
+          ixx="0.0846" ixy="0.0" ixz="0.0"
+          iyy="0.0846" iyz="0.0"
+          izz="0.0025"/>
+    </inertial>
   </link>
   <joint name="joint2" type="continuous">
@@ -115,5 +117,5 @@
     <origin xyz="0 ${-width} ${height2 - axel_offset*2}" rpy="0 0 0"/>
     <axis xyz="0 1 0"/>
-    <dynamics damping="0.7"/>
+    <dynamics damping="${damping}"/>
   </joint>
   <!-- Middle Link -->
@@ -136,8 +138,8 @@
       <mass value="${mass}"/>
       <inertia
-          ixx="${mass / 12.0 * (width*width + height3*height3)}" ixy="0.0" ixz="0.0"
-          iyy="${mass / 12.0 * (height3*height3 + width*width)}" iyz="0.0"
-          izz="${mass / 12.0 * (width*width + width*width)}"/>
-      </inertial>
+          ixx="0.0846" ixy="0.0" ixz="0.0"
+          iyy="0.0846" iyz="0.0"
+          izz="0.0025"/>
+    </inertial>
   </link>
   <joint name="joint3" type="continuous">
@@ -146,5 +148,5 @@
     <origin xyz="0 ${width} ${height3 - axel_offset*2}" rpy="0 0 0"/>
     <axis xyz="0 1 0"/>
-    <dynamics damping="0.7"/>
+    <dynamics damping="${damping}"/>
   </joint>
   <!-- First Top Link -->
@@ -167,8 +169,8 @@
       <mass value="${mass}"/>
       <inertia
-          ixx="${mass / 12.0 * (width*width + height4*height4)}" ixy="0.0" ixz="0.0"
-          iyy="${mass / 12.0 * (height4*height4 + width*width)}" iyz="0.0"
-          izz="${mass / 12.0 * (width*width + width*width)}"/>
-      </inertial>
+          ixx="0.0846" ixy="0.0" ixz="0.0"
+          iyy="0.0846" iyz="0.0"
+          izz="0.0025"/>
+    </inertial>
   </link>
   <joint name="joint4" type="continuous">
@@ -177,5 +179,5 @@
     <origin xyz="0 ${-width} ${height3 - axel_offset*2}" rpy="0 0 0"/>
     <axis xyz="0 1 0"/>
-    <dynamics damping="0.7"/>
+    <dynamics damping="${damping}"/>
   </joint>
   <!-- Second Top Link -->
@@ -198,8 +200,8 @@
       <mass value="${mass}"/>
       <inertia
-          ixx="${mass / 12.0 * (width*width + height5*height5)}" ixy="0.0" ixz="0.0"
-          iyy="${mass / 12.0 * (height5*height5 + width*width)}" iyz="0.0"
-          izz="${mass / 12.0 * (width*width + width*width)}"/>
-      </inertial>
+          ixx="0.0846" ixy="0.0" ixz="0.0"
+          iyy="0.0846" iyz="0.0"
+          izz="0.0025"/>
+    </inertial>
   </link>
   <!-- Motors so we can actuate the joints -->

Commit message: cleanup

File: multilink_balancer_description/urdf/multilink_balancer.xacro (robot description, xacro)
@@ -14,5 +14,5 @@
   <xacro:property name="foot_width" value="1.0" />
   <xacro:property name="foot_mass" value="1.0" /> <!-- negligible mass for the foot -->
-  <xacro:property name="damping" value="0.0" />
+  <xacro:property name="damping" value="0.1" />
   <xacro:property name="axel_offset" value="0.05" /> <!-- How far keep joints away from each other -->
   <!-- Import all Gazebo-customization elements, including Gazebo colors -->

Commit message: add humanoid model

File: multilink_balancer_description/urdf/multilink_balancer.xacro (robot description, xacro)
@@ -9,5 +9,5 @@
   <xacro:property name="height2" value="1.1" /> <!-- Link 2 -->
   <xacro:property name="height3" value="1.1" /> <!-- Link 3 -->
-  <xacro:property name="height4" value="1.1" /> <!-- Link 4 -->
+  <xacro:property name="height4" value="2.1" /> <!-- Link 4 -->
   <xacro:property name="height5" value="1.1" /> <!-- Link 5 -->
   <xacro:property name="foot_height" value="0.05" /> <!-- Foot dimensions -->
@@ -150,5 +150,5 @@
     <dynamics damping="${damping}"/>
   </joint>
-  <!-- First Top Link -->
+  <!-- Torso Link -->
   <link name="link4">
     <collision>
@@ -167,5 +167,5 @@
     <inertial>
       <origin xyz="0 0 ${height4/2 - axel_offset}" rpy="0 0 0"/>
-      <mass value="${mass}"/>
+      <mass value="${2*mass}"/>
       <inertia
           ixx="0.0846" ixy="0.0" ixz="0.0"
@@ -175,5 +175,5 @@
   </link>
   <joint name="joint4" type="continuous">
-    <parent link="link3"/>
+    <parent link="link4"/>
     <child link="link5"/>
     <origin xyz="0 ${-width} ${height3 - axel_offset*2}" rpy="0 0 0"/>
@@ -181,5 +181,5 @@
     <dynamics damping="${damping}"/>
   </joint>
-  <!-- Second Top Link -->
+  <!-- Arm Link -->
   <link name="link5">
     <collision>

Commit message: increase foot mass to stabilize strange noise in simulation

File: multilink_balancer_description/urdf/multilink_balancer.xacro (robot description, xacro)
@@ -13,6 +13,6 @@
   <xacro:property name="foot_height" value="0.05" /> <!-- Foot dimensions -->
   <xacro:property name="foot_width" value="1.0" />
-  <xacro:property name="foot_mass" value="1.0" /> <!-- negligible mass for the foot -->
-  <xacro:property name="damping" value="0.1" />
+  <xacro:property name="foot_mass" value="10.0" />
+  <xacro:property name="damping" value="0.0" />
   <xacro:property name="axel_offset" value="0.05" /> <!-- How far keep joints away from each other -->
   <!-- Import all Gazebo-customization elements, including Gazebo colors -->
